Commit message: CHANGE TO ROS2_CONTROL

File: amr_description/urdf/amr.urdf.xacro (robot description, xacro)
@@ -2,9 +2,17 @@
 <robot xmlns:xacro="http://www.ros.org/wiki/xacro" name="amr">
     <xacro:include filename="amr_core.xacro"/>
-    <xacro:include filename="gazebo_control.xacro"/>
-    <!-- <xacro:include filename="lidar.xacro"/> -->
+    <!-- <xacro:include filename="gazebo_control.xacro"/> -->
+    <xacro:include filename="ros2_control.xacro"/>
+    <!-- Lidar -->
     <xacro:include filename="$(find velodyne_description)/urdf/VLP-16.urdf.xacro"/>
     <xacro:VLP-16 parent="chassis" name="lidar_frame" topic="/scan" organize_cloud="false" hz="10" samples="440"  max_range="3" gpu="true">
       <origin xyz="0.73 0 0.825" rpy="0 0 0" />
     </xacro:VLP-16>
+    <!-- ARM -->
+    <!-- <xacro:include filename="$(find tm_description)/xacro/tm5-900.urdf.xacro"/>
+    <joint name="chassis_base_link" type="fixed">
+      <parent link="chassis"/>
+      <child link="base"/>
+      <origin xyz="0.37 -0.14 0.69" rpy="0 0 ${pi/2}" />
+    </joint> -->
 </robot>

File: amr_description/urdf/amr_core.xacro (robot description, xacro)
@@ -59,5 +59,5 @@
             </geometry>
         </collision>
-        <xacro:inertial_cylinder mass="0.1" length="0.04" radius="0.05">
+        <xacro:inertial_cylinder mass="0.2" length="0.04" radius="0.05">
             <origin xyz="0 0 0" rpy="0 0 0"/>
         </xacro:inertial_cylinder>
@@ -87,5 +87,5 @@
             </geometry>
         </collision>
-        <xacro:inertial_cylinder mass="0.1" length="0.04" radius="0.05">
+        <xacro:inertial_cylinder mass="0.2" length="0.04" radius="0.05">
             <origin xyz="0 0 0" rpy="0 0 0"/>
         </xacro:inertial_cylinder>
@@ -112,5 +112,5 @@
             </geometry>
         </collision>
-        <xacro:inertial_sphere mass="0.1" radius="0.05">
+        <xacro:inertial_sphere mass="0.2" radius="0.05">
             <origin xyz="0 0 0" rpy="0 0 0"/>
         </xacro:inertial_sphere>

File: tm_description/xacro/macro.gazebo.xacro (robot description, xacro)
@@ -2,28 +2,42 @@
 <robot xmlns:xacro="http://www.ros.org/wiki/xacro">
   <xacro:macro name="tmr_gazebo" params="ns prefix">
-    <gazebo reference="${prefix}link_1">
-      <selfCollide>true</selfCollide>
-    </gazebo>
-    <gazebo reference="${prefix}link_2">
-      <selfCollide>true</selfCollide>
-    </gazebo>
-    <gazebo reference="${prefix}link_3">
-      <selfCollide>true</selfCollide>
-    </gazebo>
-    <gazebo reference="${prefix}link_4">
-      <selfCollide>true</selfCollide>
-    </gazebo>
-    <gazebo reference="${prefix}link_5">
-      <selfCollide>true</selfCollide>
-    </gazebo>
-    <gazebo reference="${prefix}link_6">
-      <selfCollide>true</selfCollide>
-    </gazebo>
-    <gazebo>
-      <plugin name="gazebo_ros_control" filename="libgazebo_ros_control.so">
-        <robotNamespace>/${ns}</robotNamespace>
-        <robotSimType>gazebo_ros_control/DefaultRobotHWSim</robotSimType>
-      </plugin>
-    </gazebo>
+  <gazebo reference="base">
+    <selfCollide>true</selfCollide>
+    <material>Gazebo/Grey</material>
+  </gazebo>
+  <gazebo reference="link_0">
+    <selfCollide>true</selfCollide>
+    <material>Gazebo/Grey</material>
+  </gazebo>
+  <gazebo reference="link_1">
+    <selfCollide>true</selfCollide>
+    <material>Gazebo/Motorway</material>
+  </gazebo>
+  <gazebo reference="link_2">
+    <selfCollide>true</selfCollide>
+    <material>Gazebo/Motorway</material>
+  </gazebo>
+  <gazebo reference="link_3">
+    <selfCollide>true</selfCollide>
+    <material>Gazebo/Motorway</material>
+  </gazebo>
+  <gazebo reference="link_4">
+    <selfCollide>true</selfCollide>
+    <material>Gazebo/Motorway</material>
+  </gazebo>
+  <gazebo reference="link_5">
+    <selfCollide>true</selfCollide>
+    <material>Gazebo/Motorway</material>
+  </gazebo>
+  <gazebo reference="link_6">
+    <selfCollide>true</selfCollide>
+    <material>Gazebo/Grey</material>
+  </gazebo>
+  <gazebo>
+    <plugin name="gazebo_ros2_control" filename="libgazebo_ros2_control.so">
+      <robotNamespace>/${ns}</robotNamespace>
+      <robotSimType>gazebo_ros2_control/DefaultRobotHWSim</robotSimType>
+    </plugin>
+  </gazebo>
   </xacro:macro>
 </robot>

File: tm_description/xacro/macro.materials.xacro (robot description, xacro)
@@ -11,7 +11,7 @@
 			<color rgba="0.75 0.75 0.75 1.0" />
 		</material>
-		<material name="white">
+		<!-- <material name="white">
 			<color rgba="0.95 0.95 0.95 1.0" />
-		</material>
+		</material> -->
 		<material name="red">
 			<color rgba="0.95 0.0 0.0 1.0" />
@@ -35,7 +35,7 @@
 			<color rgba="0.6 0.0 1.0 1.0" />
 		</material>
-		<material name="black">
+		<!-- <material name="black">
 			<color rgba="0.0 0.0 0.0 1.0" />
-		</material>
+		</material> -->
 		<material name="darkolive">
 			<color rgba="0.3 0.3 0.25 1.0" />

Commit message: some ros2 control changes

File: amr_description/urdf/amr.urdf.xacro (robot description, xacro)
@@ -1,7 +1,12 @@
 <?xml version="1.0"?>
 <robot xmlns:xacro="http://www.ros.org/wiki/xacro" name="amr">
+    <xacro:arg name="use_ros2_control" default="true"/>
     <xacro:include filename="amr_core.xacro"/>
-    <!-- <xacro:include filename="gazebo_control.xacro"/> -->
-    <xacro:include filename="ros2_control.xacro"/>
+    <xacro:if value="$(arg use_ros2_control)">
+      <xacro:include filename="ros2_control.xacro" />
+    </xacro:if>
+    <xacro:unless value="$(arg use_ros2_control)">
+      <xacro:include filename="gazebo_control.xacro" />
+    </xacro:unless>
     <!-- Lidar -->
     <xacro:include filename="$(find velodyne_description)/urdf/VLP-16.urdf.xacro"/>

File: amr_description/urdf/amr_core.xacro (robot description, xacro)
@@ -31,5 +31,5 @@
             </geometry>
         </collision>
-        <xacro:inertial_box mass="40" x="0.96" y="0.46" z="0.69">
+        <xacro:inertial_box mass="0.5" x="0.96" y="0.46" z="0.69">
             <origin xyz="0.48 0.0 0.345" rpy="0 0 0"/>
         </xacro:inertial_box>
@@ -56,5 +56,5 @@
             <origin xyz="0.0 0.0 0.0" rpy="0.0 0.0 0.0"/>
             <geometry>
-                <cylinder radius="0.05" length="0.04"/>
+                <sphere radius="0.05" />
             </geometry>
         </collision>
@@ -84,5 +84,5 @@
             <origin xyz="0.0 0.0 0.0" rpy="0.0 0.0 0.0"/>
             <geometry>
-                <cylinder radius="0.05" length="0.04"/>
+                <sphere radius="0.05" />
             </geometry>
         </collision>

Commit message: 20230322

File: amr_description/urdf/amr.urdf.xacro (robot description, xacro)
@@ -11,5 +11,5 @@
     <!-- Lidar -->
     <xacro:include filename="$(find velodyne_description)/urdf/VLP-16.urdf.xacro"/>
-    <xacro:VLP-16 parent="chassis" name="lidar_frame" topic="/scan" organize_cloud="false" hz="10" samples="440"  max_range="3" gpu="true">
+    <xacro:VLP-16 parent="chassis" name="lidar_frame" topic="/velodyne" organize_cloud="false" hz="10" samples="440"  max_range="3" gpu="true">
       <origin xyz="0.73 0 0.825" rpy="0 0 0" />
     </xacro:VLP-16>

File: amr_description/urdf/amr_core.xacro (robot description, xacro)
@@ -10,4 +10,12 @@
     <!-- BASE_LINK -->
     <link name="base_link">
+    </link>
+    <!-- BASE_FOOTPRINT LINK -->
+    <joint name="base_footprint_joint" type="fixed">
+        <parent link="base_link"/>
+        <child link="base_footprint"/>
+        <origin xyz="0.0 0.0 0.0" rpy="0 0 0"/>
+    </joint>
+    <link name="base_footprint">
     </link>
     <!-- CHASSIS_LINK -->
